File: schematics/gp5.sch (EAGLE design)
At the start: 11 parts, among them IC1 317T, IC2 317EMP, IC3 TLE5205-2S

Commit message: finalised schematic files
Parts:
- removed IC3: TLE5205-2S, infineon:TLE5205-2S
- removed JP2: (no value), pinhead:PINHD-1X3
- removed JP3: (no value), pinhead:PINHD-2X3
- removed JP4: (no value), pinhead:PINHD-2X8
- added JP5: (no value), pinhead:PINHD-2X7
- JP1: device pinhead:PINHD-1X2 -> pinhead:PINHD-2X3
Connections:
- removed net MOTOR_OUT1: IC3.OUT1, JP1.1
- removed net N$2: IC3.OUT2, JP1.2
- removed net N$3: IC3.EF, JP2.3
- removed net N$4: IC3.IN1, JP2.2
- removed net N$5: IC3.IN2, JP2.1
- net +3.3V: now also JP5.10, JP5.12, JP5.14, JP5.2, JP5.4, JP5.6, JP5.8; no longer JP3.2, JP3.4, JP3.6
- net +5V_R: now also JP1.2, JP1.4, JP1.6; no longer IC3.VS, JP4.10, JP4.12, JP4.14, JP4.16, JP4.2, JP4.4, JP4.6, JP4.8
- net GND: now also JP1.1, JP1.3, JP1.5, JP5.1, JP5.11, JP5.13, JP5.3, JP5.5, JP5.7, JP5.9; no longer IC3.GND, JP3.1, JP3.3, JP3.5, JP4.1, JP4.11, JP4.13, JP4.15, JP4.3, JP4.5, JP4.7, JP4.9
